Commit message: refactor: move sdf to dedicated folder

File: embodiment_assets/skeleton.urdf (robot description, URDF)
Before this commit: robot skeleton, 10 links, 9 joints
Links:
- link skeleton__distal: geometry collision mesh filename=package://meshes/distal.obj scale=1.0 1.0 1.0; visual mesh filename=package://meshes/distal.obj scale=1.0 1.0 1.0
- link skeleton__forearm: geometry collision mesh filename=package://meshes/forearm.obj scale=1.0 1.0 1.0; visual mesh filename=package://meshes/forearm.obj scale=1.0 1.0 1.0
- link skeleton__hand: geometry collision mesh filename=package://meshes/hand_col.dae scale=1.0 1.0 1.0; visual mesh filename=package://meshes/hand.obj scale=1.0 1.0 1.0
- link skeleton__middle: geometry collision mesh filename=package://meshes/middle_col.dae scale=1.0 1.0 1.0; visual mesh filename=package://meshes/middle.obj scale=1.0 1.0 1.0
- link skeleton__proximal: geometry collision mesh filename=package://meshes/proximal_col.dae scale=1.0 1.0 1.0; visual mesh filename=package://meshes/proximal.obj scale=1.0 1.0 1.0
- link skeleton__thumb_1: geometry visual mesh filename=package://meshes/thumb_1.obj scale=1.0 1.0 1.0
- link skeleton__thumb_2: geometry visual mesh filename=package://meshes/thumb_2.obj scale=1.0 1.0 1.0
- link skeleton__thumb_3: geometry visual mesh filename=package://meshes/thumb_3.obj scale=1.0 1.0 1.0
- link skeleton__upper_arm: geometry collision mesh filename=package://meshes/upper_arm.obj scale=1.0 1.0 1.0; visual mesh filename=package://meshes/upper_arm.obj scale=1.0 1.0 1.0
