Commit message: feat: move shoulder initial pos to manipulandum setup

File: src/neurocontroller/embodiment_assets/skeleton.urdf (robot description, URDF)
Before this commit: robot skeleton, 10 links, 9 joints
Joints:
- joint skeleton__shoulder_joint: axis 1 0 0 -> 0 -0.17364817766693033 0.984807753012208; limit lower=-1 upper=0.7853981852531433 effort=0.0 velocity=0.0 -> lower=-1.5707963705062866 upper=1.5707963705062866 effort=0.0 velocity=0.0; origin xyz=-0.01754 -0.17     1.793 rpy=1.59151 1.57079 0.02072 -> xyz=-0.01754 -0.17     1.793 rpy=-0.17453292519943295 0 0
